Commit message: new stuff

File: catbot_pybullet/meshes/catbot.urdf (robot description, URDF)
Before this commit: robot catbot.urdf, 13 links, 12 joints
Links:
- link botlegasm: mass 0.054645620986758416948 -> 0.0546456; geometry collision mesh filename=package://catbot_pybullet/meshes/botleg.stl; collision mesh filename=package://catbot_pybullet/meshes/servo.stl
- link botlegasm_2: mass 0.054645620986758416948 -> 0.0546456; geometry collision mesh filename=package://catbot_pybullet/meshes/botleg.stl; collision mesh filename=package://catbot_pybullet/meshes/servo.stl
- link botlegasm_3: mass 0.054645620986758416948 -> 0.0546456; geometry collision mesh filename=package://catbot_pybullet/meshes/botleg.stl; collision mesh filename=package://catbot_pybullet/meshes/servo.stl
- link botlegasm_4: mass 0.054645620986758416948 -> 0.0546456; geometry collision mesh filename=package://catbot_pybullet/meshes/botleg.stl; collision mesh filename=package://catbot_pybullet/meshes/servo.stl
- link hipsubasm: mass 0.066123103332140956145 -> 0.0661231; geometry collision mesh filename=package://catbot_pybullet/meshes/hipjoint.stl; collision mesh filename=package://catbot_pybullet/meshes/servo.stl
- link hipsubasm_2: mass 0.066123103332140956145 -> 0.0661231; geometry collision mesh filename=package://catbot_pybullet/meshes/hipjoint.stl; collision mesh filename=package://catbot_pybullet/meshes/servo.stl
- link mainbody: mass 0.49394823622559713705 -> 0.493948; geometry collision mesh filename=package://catbot_pybullet/meshes/base.stl; collision mesh filename=package://catbot_pybullet/meshes/servo.stl
- link mirroredhipsubasm: mass 0.066123103332140956145 -> 0.0661231; geometry collision mesh filename=package://catbot_pybullet/meshes/mirrorhipjoint.stl; collision mesh filename=package://catbot_pybullet/meshes/servo.stl
- link mirroredhipsubasm_2: mass 0.066123103332140956145 -> 0.0661231; geometry collision mesh filename=package://catbot_pybullet/meshes/mirrorhipjoint.stl; collision mesh filename=package://catbot_pybullet/meshes/servo.stl
- link toplegasm: mass 0.025684018857765292254 -> 0.025684; geometry collision mesh filename=package://catbot_pybullet/meshes/servohornreplacement.stl; collision mesh filename=package://catbot_pybullet/meshes/servohornreplacement.stl
- link toplegasm_2: mass 0.025684018857765292254 -> 0.025684; geometry collision mesh filename=package://catbot_pybullet/meshes/servohornreplacement.stl; collision mesh filename=package://catbot_pybullet/meshes/servohornreplacement.stl
- link toplegasm_3: mass 0.025684018857765292254 -> 0.025684; geometry collision mesh filename=package://catbot_pybullet/meshes/servohornreplacement.stl; collision mesh filename=package://catbot_pybullet/meshes/servohornreplacement.stl
- link toplegasm_4: mass 0.025684018857765292254 -> 0.025684; geometry collision mesh filename=package://catbot_pybullet/meshes/servohornreplacement.stl; collision mesh filename=package://catbot_pybullet/meshes/servohornreplacement.stl
Joints:
- joint BL_BotLeg: limit effort=1 velocity=20 -> lower=-3.141592653589793 upper=3.141592653589793 effort=10 velocity=10; origin xyz=1.9428902930940239457e-16 0.11200000000000062683 3.8857805861880478915e-16 rpy=3.1415926535897926719 -1.0243549092722601103e-15 3.1262445307774839875 -> xyz=0 0.112 -0 rpy=-3.14159 0 1.5708
- joint BL_Hip: limit lower=-0.785398163397448279 upper=0.785398163397448279 effort=1 velocity=20 -> lower=-0.785398 upper=0.785398 effort=10 velocity=10; origin xyz=-0.17420040591955210374 -0.18684034999608997718 0.23555598676204667075 rpy=-1.57079632679489678 0.0117328984293165791 1.2601170739682348073e-15 -> xyz=-0 -0 0.16305 rpy=3.14159 -0 -0
- joint BL_TopLeg: limit lower=-1.570796326794896558 upper=1.570796326794896558 effort=1 velocity=20 -> lower=-1.5708 upper=1.5708 effort=10 velocity=10; origin xyz=-0.022250000000000019762 0.02826499999999992907 -0.020000000000000017764 rpy=1.0152967728242205898e-15 1.5707963267948952257 0 -> xyz=-0.02225 0.028265 -0.02 rpy=0 1.5708 0
- joint BR_BotLeg: limit effort=1 velocity=20 -> lower=-3.141592653589793 upper=3.141592653589793 effort=10 velocity=10; origin xyz=-2.7755575615628913511e-17 0.11199999999999990519 5.5511151231257827021e-17 rpy=-3.1415926535897886751 -7.0938256185667662878e-15 0.58170270124798439948 -> xyz=-0 0.112 0 rpy=3.14159 -0 1.5708
- joint BR_Hip: child hipsubasm -> hipsubasm_2; limit lower=-0.785398163397448279 upper=0.785398163397448279 effort=1 velocity=20 -> lower=-0.785398 upper=0.785398 effort=10 velocity=10; origin xyz=-0.063900405919551844791 -0.18684034999608994942 0.23555598676204686504 rpy=1.570796326794896558 -0.041547970194335065441 3.141592653589793116 -> xyz=0.1103 -0 0.16305 rpy=-3.14159 0 3.14159
- joint BR_TopLeg: limit lower=-1.570796326794896558 upper=1.570796326794896558 effort=1 velocity=20 -> lower=-1.5708 upper=1.5708 effort=10 velocity=10; origin xyz=-0.022249999999999943434 -0.028264999999999401714 -0.019999999999999990008 rpy=-1.5707963267948958919 -1.5476780753609129526 -1.5707963267949160979 -> xyz=-0.02225 -0.028265 -0.02 rpy=3.14159 -1.5708 0; parent hipsubasm -> hipsubasm_2
- joint FL_BotLeg: limit effort=1 velocity=20 -> lower=-3.141592653589793 upper=3.141592653589793 effort=10 velocity=10; origin xyz=4.1633363423443370266e-17 0.11199999999999782352 -1.3322676295501878485e-15 rpy=-3.1415926535897784611 4.6425528594852074692e-15 2.9239169939649158891 -> xyz=0 0.112 -0 rpy=3.14159 0 1.5708
- joint FL_Hip: child hipsubasm_2 -> mainbody; limit lower=-0.785398163397448279 upper=0.785398163397448279 effort=1 velocity=20 -> lower=-0.785398 upper=0.785398 effort=10 velocity=10; origin xyz=-0.17420040591955185394 -0.023790349996089921181 0.23555598676204680952 rpy=1.570796326794896558 0.053772588985834847419 2.2234000273411940108e-16 -> xyz=-0.1742 -0.0237903 0.235556 rpy=1.5708 -0 0; parent mainbody -> hipsubasm
- joint FL_TopLeg: limit lower=-1.570796326794896558 upper=1.570796326794896558 effort=1 velocity=20 -> lower=-1.5708 upper=1.5708 effort=10 velocity=10; origin xyz=-0.022249999999999825473 -0.028264999999999845803 -0.020000000000000003886 rpy=1.570796326794896558 -1.4084388595620607187 1.5707963267949249797 -> xyz=-0.19645 -0.00379035 0.207291 rpy=-1.5708 0 -1.5708; parent hipsubasm_2 -> hipsubasm
- joint FR_BotLeg: limit effort=1 velocity=20 -> lower=-3.141592653589793 upper=3.141592653589793 effort=10 velocity=10; origin xyz=9.4108748571741784872e-17 0.11200000000000287503 3.0531133177191804862e-16 rpy=-3.1415926535897922278 -4.3401406628148288015e-16 -0.14343495739683284618 -> xyz=-0 0.112 0 rpy=-3.14159 -0 1.5708
- joint FR_Hip: limit lower=-0.785398163397448279 upper=0.785398163397448279 effort=1 velocity=20 -> lower=-0.785398 upper=0.785398 effort=10 velocity=10; origin xyz=-0.063900405919551941936 -0.023790349996089938528 0.23555598676204683728 rpy=-1.570796326794896558 -0.082892067804055696856 -3.141592653589793116 -> xyz=0.1103 -0 0 rpy=0 0 3.14159
- joint FR_TopLeg: limit lower=-1.570796326794896558 upper=1.570796326794896558 effort=1 velocity=20 -> lower=-1.5708 upper=1.5708 effort=10 velocity=10; origin xyz=-0.022250000000000103029 0.028265000000000067848 -0.020000000000000007355 rpy=-2.696149045489602097e-16 1.5707963267948956698 0 -> xyz=-0.02225 0.028265 -0.02 rpy=-0 1.5708 0
